File: sch/squid.kicad_pcb (KiCad board)
At the start: 2 copper layers, 177.3 x 205 mm, 51 parts, among them IC1 MAX3241, IC2 MAX3241, IC3 MAX3241, J10 BOXHDR2x3, J3 BOXHDR2x5, J4 BOXHDR2x5, J6 BOXHDR2x5, J8 BOXHDR2x5, J9 CONN_01X06, P1 CONN_01X06, P11 CONN_01X04, P2 USB_OTG, P3 CONN_02X10, P4 CONN_01X10, P5 CONN_01X06, P6 TERM_BLOCK_1x5, P8 CONN_01X10, P9 CONN_01X06, U1 LPC1769FBD100, U10 74HC595, U11 74HC595, U12 74HC595, U2 FT232RL, U3 74xx125, U4 74xx125, U5 74xx125, U6 75LBC176, U7 75LBC176, U8 74xx125, U9 74HC595

Commit message: Draft 1, PCB Preliminary Placement
Parts:
- removed IC1, IC2, IC3: MAX3241, Housings_SSOP:SSOP-28_5.3x10.2mm_Pitch0.65mm
- removed JP1, JP2: JUMPER3, Pin_Headers:Pin_Header_Straight_1x03
- removed P1, P5, P9: CONN_01X06, Pin_Headers:Pin_Header_Straight_1x06
- removed P11: CONN_01X04, Pin_Headers:Pin_Header_Straight_1x04
- removed P2: USB_OTG, Connect:USB_Micro-B
- removed P3: CONN_02X10, Pin_Headers:Pin_Header_Straight_2x10
- removed P4, P8: CONN_01X10, Pin_Headers:Pin_Header_Straight_1x10
- removed P6: TERM_BLOCK_1x5, TERM-STRIP-5
- added C13: 18pF, Capacitors_SMD:C_0805_HandSoldering, F.Cu at (0.50, 89.8)
- added C14: 0.1uF, Capacitors_SMD:C_0805_HandSoldering, F.Cu at (52.7, 103.2)
- added C15: 0.1uF, Capacitors_SMD:C_0805_HandSoldering, F.Cu at (52.7, 115.2)
- added C16: 0.1uF, Capacitors_SMD:C_0805_HandSoldering, F.Cu at (54.2, 130.9)
- added C17: 0.1uF, Capacitors_SMD:C_0805_HandSoldering, F.Cu at (54.7, 115.2)
- added C18: 0.1uF, Capacitors_SMD:C_0805_HandSoldering, F.Cu at (52.2, 130.9)
- added C19: 0.47uF, Capacitors_SMD:C_0805_HandSoldering, F.Cu at (-10.5, 148.2)
- added C20: 0.47uF, Capacitors_SMD:C_0805_HandSoldering, F.Cu at (-10.5, 135.2)
- added C21: 0.1uF, Capacitors_SMD:C_0805_HandSoldering, F.Cu at (41.0, 176.8)
- added C22: 10uF, Capacitors_Tantalum_SMD:TantalC_SizeB_EIA-3528_HandSoldering, F.Cu at (55.1, 187.8)
- added C23: 0.1uF, Capacitors_SMD:C_0805_HandSoldering, F.Cu at (77.8, 161.5)
- added C24: 0.1uF, Capacitors_SMD:C_0805_HandSoldering, F.Cu at (79.8, 155.8)
- added C25: 0.1uF, Capacitors_SMD:C_0805_HandSoldering, F.Cu at (78.5, 159.6)
- added C26: 0.1uF, Capacitors_SMD:C_0805_HandSoldering, F.Cu at (79.2, 157.7)
- added C27: 1.0uF, Capacitors_SMD:C_0805_HandSoldering, F.Cu at (53.3, 50.1)
- added C28: 10uF, Capacitors_Tantalum_SMD:TantalC_SizeB_EIA-3528_HandSoldering, F.Cu at (57.8, 54.2)
- added C29: 0.1uF, Capacitors_SMD:C_0805_HandSoldering, F.Cu at (-31.9, 180.5)
- added C30: 0.1uF, Capacitors_SMD:C_0805_HandSoldering, F.Cu at (34.8, 203.9)
- added C31: 0.1uF, Capacitors_SMD:C_0805_HandSoldering, F.Cu at (-32.7, 204.2)
- added C32: 0.1uF, Capacitors_SMD:C_0805_HandSoldering, F.Cu at (-40.2, 148.5)
- added C33: 0.1uF, Capacitors_SMD:C_0805_HandSoldering, F.Cu at (-40.0, 139.2)
- added C34: 0.1uF, Capacitors_SMD:C_0805_HandSoldering, F.Cu at (-37.0, 129.8)
- added C35: 0.1uF, Capacitors_SMD:C_0805_HandSoldering, F.Cu at (-24.5, 159.0)
- added C36: 0.1uF, Capacitors_SMD:C_0805_HandSoldering, F.Cu at (-5.75, 164.5)
- added C37: 0.1uF, Capacitors_SMD:C_0805_HandSoldering, F.Cu at (12.2, 164.0)
- added C38: 0.1uF, Capacitors_SMD:C_0805_HandSoldering, F.Cu at (28.0, 158.5)
- added C39: 1.0uF, Capacitors_SMD:C_0805_HandSoldering, F.Cu at (-14.2, 102.0)
- added C40: 0.1uF, Capacitors_SMD:C_0805_HandSoldering, F.Cu at (-4.25, 119.5)
- added C41: 0.1uF, Capacitors_SMD:C_0805_HandSoldering, F.Cu at (4.25, 119.5)
- added C42: 0.1uF, Capacitors_SMD:C_0805_HandSoldering, F.Cu at (14.2, 103.0)
- added C43: 0.1uF, Capacitors_SMD:C_0805_HandSoldering, F.Cu at (14.2, 109.0)
- added C44: 0.1uF, Capacitors_SMD:C_0805_HandSoldering, F.Cu at (-14.2, 109.0)
- added C45: 0.1uF, Capacitors_SMD:C_0805_HandSoldering, F.Cu at (6.75, 92.5)
- added C46: 0.1uF, Capacitors_SMD:C_0805_HandSoldering, F.Cu at (38.0, 105.7)
- added C47: 0.1uF, Capacitors_SMD:C_0805_HandSoldering, F.Cu at (28.0, 115.2)
- added C48: 0.1uF, Capacitors_SMD:C_0805_HandSoldering, F.Cu at (50.7, 115.2)
- added C49: 0.1uF, Capacitors_SMD:C_0805_HandSoldering, F.Cu at (38.0, 100.7)
- added C50: 0.1uF, Capacitors_SMD:C_0805_HandSoldering, F.Cu at (28.0, 131.2)
- added C51: 0.1uF, Capacitors_SMD:C_0805_HandSoldering, F.Cu at (26.8, 75.5)
- added C52: 0.1uF, Capacitors_SMD:C_0805_HandSoldering, F.Cu at (10.5, 142.2)
- added C53: 0.1uF, Capacitors_SMD:C_0805_HandSoldering, F.Cu at (10.5, 144.2)
- added C54: 0.1uF, Capacitors_SMD:C_0805_HandSoldering, F.Cu at (52.5, 170.8)
- added C55: 0.1uF, Capacitors_SMD:C_0805_HandSoldering, F.Cu at (52.5, 160.7)
- added C56: 0.1uF, Capacitors_SMD:C_0805_HandSoldering, F.Cu at (63.8, 165.8)
- added C57: 0.1uF, Capacitors_SMD:C_0805_HandSoldering, F.Cu at (55.1, 153.6)
- added C58: 0.1uF, Capacitors_SMD:C_0805_HandSoldering, F.Cu at (63.1, 149.1)
- added C59: 10uF, Capacitors_Tantalum_SMD:TantalC_SizeB_EIA-3528_HandSoldering, F.Cu at (62.8, 145.0)
- added C60: 0.1uF, Capacitors_SMD:C_0805_HandSoldering, F.Cu at (44.8, 165.7)
- added C61: 0.1uF, Capacitors_SMD:C_0805_HandSoldering, F.Cu at (39.3, 175.6)
- added C62: 0.1uF, Capacitors_SMD:C_0805_HandSoldering, F.Cu at (58.4, 50.1)
- added C63: 0.1uF, Capacitors_SMD:C_0805_HandSoldering, F.Cu at (-43.5, 32.5)
- added C64: 0.1uF, Capacitors_SMD:C_0805_HandSoldering, F.Cu at (18.0, 194.9)
- added C65: 0.1uF, Capacitors_SMD:C_0805_HandSoldering, F.Cu at (6.12, 196.5)
- added C66: 0.1uF, Capacitors_SMD:C_0805_HandSoldering, F.Cu at (-15.2, 188.7)
- added C67: 0.1uF, Capacitors_SMD:C_0805_HandSoldering, F.Cu at (23.9, 210.2)
- added C68: 0.1uF, Capacitors_SMD:C_0805_HandSoldering, F.Cu at (6.49, 213.9)
- added C69: 0.1uF, Capacitors_SMD:C_0805_HandSoldering, F.Cu at (-6.58, 210.9)
- added D1: LED-GREEN, Resistors_SMD:R_0805_HandSoldering, F.Cu at (-6.58, 207.7)
- added D10: LED-GREEN, Resistors_SMD:R_0805_HandSoldering, F.Cu at (-56.5, 120.2)
- added D11: LED-GREEN, Resistors_SMD:R_0805_HandSoldering, F.Cu at (-56.5, 105.5)
- added D12: LED-GREEN, Resistors_SMD:R_0805_HandSoldering, F.Cu at (-77.0, 156.7)
- added D13: LED-GREEN, Resistors_SMD:R_0805_HandSoldering, F.Cu at (-62.9, 151.6)
- added D14: LED-GREEN, Resistors_SMD:R_0805_HandSoldering, F.Cu at (-54.7, 185.1)
- added D15: LED-GREEN, Resistors_SMD:R_0805_HandSoldering, F.Cu at (-45.2, 173.8)
- added D16: LED-GREEN, Resistors_SMD:R_0805_HandSoldering, F.Cu at (-63.6, 174.2)
- added D17: LED-GREEN, Resistors_SMD:R_0805_HandSoldering, F.Cu at (-56.5, 126.5)
- added D18: LED-GREEN, Resistors_SMD:R_0805_HandSoldering, F.Cu at (48.7, 115.2)
- added D19: LED-GREEN, Resistors_SMD:R_0805_HandSoldering, F.Cu at (42.7, 115.2)
- added D2: LED-GREEN, Resistors_SMD:R_0805_HandSoldering, F.Cu at (-6.58, 192.9)
- added D20: LED-GREEN, Resistors_SMD:R_0805_HandSoldering, F.Cu at (54.7, 103.2)
- added D21: 1N4148, Diodes_SMD:SOD-123, F.Cu at (0.00, 23.8)
- added D22: 1N4148, Diodes_SMD:SOD-123, F.Cu at (22.5, 23.8)
- added D23: 1N4148, Diodes_SMD:SOD-123, F.Cu at (-7.50, 23.8)
- added D24: 1N4148, Diodes_SMD:SOD-123, F.Cu at (15.0, 23.8)
- added D25: 1N4148, Diodes_SMD:SOD-123, F.Cu at (-15.0, 23.8)
- added D26: 1N4148, Diodes_SMD:SOD-123, F.Cu at (-22.5, 23.8)
- added D27: 1N4148, Diodes_SMD:SOD-123, F.Cu at (7.50, 23.8)
- added D28: BAT54, TO_SOT_Packages_SMD:SOT-23_Handsoldering, F.Cu at (-10.5, 140.0)
- added D29: BAT54, TO_SOT_Packages_SMD:SOT-23_Handsoldering, F.Cu at (-10.5, 143.5)
- added D3: LED-GREEN, Resistors_SMD:R_0805_HandSoldering, F.Cu at (-6.58, 188.9)
- added D30: LED-GREEN, Resistors_SMD:R_0805_HandSoldering, F.Cu at (65.3, 175.4)
- added D31: LED-GREEN, Resistors_SMD:R_0805_HandSoldering, F.Cu at (51.6, 184.2)
- added D32: LED-GREEN, Resistors_SMD:R_0805_HandSoldering, F.Cu at (59.0, 191.7)
- added D33: LED-GREEN, Resistors_SMD:R_0805_HandSoldering, F.Cu at (74.7, 182.0)
- added D34: LED-GREEN, Resistors_SMD:R_0805_HandSoldering, F.Cu at (48.4, 199.1)
- added D35: LED-GREEN, Resistors_SMD:R_0805_HandSoldering, F.Cu at (-42.4, 190.3)
- added D36: LED-GREEN, Resistors_SMD:R_0805_HandSoldering, F.Cu at (43.7, 158.5)
- added D4: LED-GREEN, Resistors_SMD:R_0805_HandSoldering, F.Cu at (-19.6, 201.1)
- added D5: LED-GREEN, Resistors_SMD:R_0805_HandSoldering, F.Cu at (6.49, 205.9)
- added D6: LED-GREEN, Resistors_SMD:R_0805_HandSoldering, F.Cu at (-31.5, 200.9)
- added D7: LED-GREEN, Resistors_SMD:R_0805_HandSoldering, F.Cu at (-26.4, 186.8)
- added D8: LED-GREEN, Resistors_SMD:R_0805_HandSoldering, F.Cu at (-25.0, 183.1)
- added D9: LED-GREEN, Resistors_SMD:R_0805_HandSoldering, F.Cu at (-86.0, 159.9)
- added DS1: LCD-4x20, my-display:NHD-0420AZ, F.Cu at (27.9, 69.8)
- added J1: HDR-1x10, my-connect:PHDR-RA-SMT-1x10, B.Cu at (-27.3, 220.0)
- added J11: HDR-1x6, my-connect:PHDR-RA-SMT-1x6, B.Cu at (-89.4, 156.1)
- added J12: BOXHDR-2x3, my-connect:SHDR-SMT-2x3, F.Cu at (-70.4, 185.8)
- added J13: BOXHDR-2x3, my-connect:SHDR-SMT-2x3, F.Cu at (-97.1, 170.2)
- added J14: HDR-1x4, my-connect:PHDR-RA-SMT-1x4, B.Cu at (-79.1, 180.5)
- added J15: BOXHDR-2x5, my-connect:SHDR-SMT-2x5, F.Cu at (75.7, 131.1)
- added J16: HDR-1x10, my-connect:PHDR-RA-SMT-1x10, B.Cu at (64.5, 128.9)
- added J17: USB-MICRO-B, Connect:USB_Micro-B, F.Cu at (76.8, 103.2)
- added J18: MINIDIN6, my-connect:MINIDIN-STR-THRU-6, F.Cu at (-101.2, 156.5)
- added J19: HDR-1x6, my-connect:PHDR-RA-SMT-1x6, B.Cu at (-43.0, 43.0)
- added J2: TERM-BLOCK-5, my-connect:term-block-5, F.Cu at (18.0, 227.3)
- added J20: BOXHDR-2x10, my-connect:SHDR-SMT-2x10, F.Cu at (-55.2, 38.0)
- added J21: RJ45-MAGS, my-connect:RJ45_TRANSFO_PULSE_A, F.Cu at (88.4, 166.7)
- added J22: USB-TYPE-A, Connect:USB_A, F.Cu at (68.5, 198.8)
- added J23: USB-MICRO-B, Connect:USB_Micro-B, F.Cu at (89.0, 189.1)
- added J24: USB-MICRO-B, Connect:USB_Micro-B, F.Cu at (43.3, 22.6)
- added J25: HDR-1x4, my-connect:PHDR-RA-SMT-1x4, B.Cu at (43.6, 212.5)
- added J5: HDR-1x10, my-connect:PHDR-RA-SMT-1x10, B.Cu at (-55.5, 205.4)
- added J7: BOXHDR-2x10, my-connect:SHDR-SMT-2x10, F.Cu at (-73.7, 104.8)
- added LS1: BUZZER, my-misc:BUZZER-CSS-0575A, F.Cu at (42.5, 41.8)
- added Q1: 2N3904, my-sot-packages:SOT-23-BEC-HAND, F.Cu at (-21.2, 205.6)
- added Q10: DMG1013, my-sot-packages:SOT-323-GSD-HAND, F.Cu at (-49.2, 178.5)
- added Q11: DMG1013, my-sot-packages:SOT-323-GSD-HAND, F.Cu at (-50.7, 180.3)
- added Q12: 2N3904, my-sot-packages:SOT-23-BEC-HAND, F.Cu at (-81.5, 158.3)
- added Q13: 2N3904, my-sot-packages:SOT-23-BEC-HAND, F.Cu at (61.5, 103.2)
- added Q14: 2N3904, my-sot-packages:SOT-23-BEC-HAND, F.Cu at (47.5, 130.9)
- added Q15: 2N3904, my-sot-packages:SOT-23-BEC-HAND, F.Cu at (38.0, 115.2)
- added Q16: 2N3904, my-sot-packages:SOT-23-BEC-HAND, F.Cu at (40.0, 130.9)
- added Q17: 2N3904, my-sot-packages:SOT-23-BEC-HAND, F.Cu at (53.5, 37.3)
- added Q18: 2N2222, my-sot-packages:SOT-23-BEC-HAND, F.Cu at (10.5, 139.5)
- added Q19: 2N3906, my-sot-packages:SOT-23-BEC-HAND, F.Cu at (69.2, 178.1)
- added Q2: DMG1013, my-sot-packages:SOT-323-GSD-HAND, F.Cu at (-6.58, 199.2)
- added Q20: 2N3904, my-sot-packages:SOT-23-BEC-HAND, F.Cu at (-45.5, 193.9)
- added Q3: DMG1013, my-sot-packages:SOT-323-GSD-HAND, F.Cu at (-6.58, 201.4)
- added Q4: DMG1013, my-sot-packages:SOT-323-GSD-HAND, F.Cu at (-28.6, 192.8)
- added Q5: DMG1013, my-sot-packages:SOT-323-GSD-HAND, F.Cu at (-29.4, 195.1)
- added Q6: DMG1013, my-sot-packages:SOT-323-GSD-HAND, F.Cu at (-56.5, 111.8)
- added Q7: DMG1013, my-sot-packages:SOT-323-GSD-HAND, F.Cu at (-68.8, 153.7)
- added Q8: DMG1013, my-sot-packages:SOT-323-GSD-HAND, F.Cu at (-56.5, 114.0)
- added Q9: DMG1013, my-sot-packages:SOT-323-GSD-HAND, F.Cu at (-71.2, 154.6)
- added R10: 10K, Resistors_SMD:R_0805_HandSoldering, F.Cu at (-6.58, 203.7)
- added R100: 10K, Resistors_SMD:R_0805_HandSoldering, F.Cu at (36.1, 173.3)
- added R101: 1K, Resistors_SMD:R_0805_HandSoldering, F.Cu at (-47.2, 196.0)
- added R102: 10K, Resistors_SMD:R_0805_HandSoldering, F.Cu at (-43.7, 191.8)
- added R103: 220, Resistors_SMD:R_0805_HandSoldering, F.Cu at (47.2, 197.6)
- added R104: 220, Resistors_SMD:R_0805_HandSoldering, F.Cu at (-41.1, 188.8)
- added R105: 10K, Resistors_SMD:R_0805_HandSoldering, F.Cu at (45.8, 152.9)
- added R106: 220, Resistors_SMD:R_0805_HandSoldering, F.Cu at (44.4, 156.7)
- added R107: 4.7K, Resistors_SMD:R_0805_HandSoldering, F.Cu at (-56.7, 170.2)
- added R108: 4.7K, Resistors_SMD:R_0805_HandSoldering, F.Cu at (-58.4, 171.2)
- added R109: 4.7K, Resistors_SMD:R_0805_HandSoldering, F.Cu at (10.5, 150.2)
- added R11: 220, Resistors_SMD:R_0805_HandSoldering, F.Cu at (-6.58, 205.7)
- added R110: 4.7K, Resistors_SMD:R_0805_HandSoldering, F.Cu at (-10.5, 150.2)
- added R12: 220, Resistors_SMD:R_0805_HandSoldering, F.Cu at (-6.58, 194.9)
- added R13: 220, Resistors_SMD:R_0805_HandSoldering, F.Cu at (-6.58, 190.9)
- added R14: 220, Resistors_SMD:R_0805_HandSoldering, F.Cu at (-18.9, 199.2)
- added R15: 220, Resistors_SMD:R_0805_HandSoldering, F.Cu at (6.49, 207.9)
- added R16: 10K, Resistors_SMD:R_0805_HandSoldering, F.Cu at (49.7, 200.7)
- added R17: 10K, Resistors_SMD:R_0805_HandSoldering, F.Cu at (-39.8, 187.2)
- added R18: 60, Resistors_SMD:R_0805_HandSoldering, F.Cu at (51.0, 202.2)
- added R19: 60, Resistors_SMD:R_0805_HandSoldering, F.Cu at (53.6, 205.3)
- added R20: 10K, Resistors_SMD:R_0805_HandSoldering, F.Cu at (-27.8, 190.6)
- added R21: 10K, Resistors_SMD:R_0805_HandSoldering, F.Cu at (-30.2, 197.2)
- added R22: 220, Resistors_SMD:R_0805_HandSoldering, F.Cu at (-30.8, 199.1)
- added R23: 220, Resistors_SMD:R_0805_HandSoldering, F.Cu at (-27.1, 188.7)
- added R24: 220, Resistors_SMD:R_0805_HandSoldering, F.Cu at (-25.7, 185.0)
- added R25: 10K, Resistors_SMD:R_0805_HandSoldering, F.Cu at (-60.1, 172.2)
- added R26: 10K, Resistors_SMD:R_0805_HandSoldering, F.Cu at (-56.5, 122.2)
- added R27: 10K, Resistors_SMD:R_0805_HandSoldering, F.Cu at (-56.5, 109.5)
- added R28: 10K, Resistors_SMD:R_0805_HandSoldering, F.Cu at (-66.7, 152.9)
- added R29: 10K, Resistors_SMD:R_0805_HandSoldering, F.Cu at (-56.5, 116.2)
- added R30: 10K, Resistors_SMD:R_0805_HandSoldering, F.Cu at (-73.3, 155.3)
- added R31: 10K, Resistors_SMD:R_0805_HandSoldering, F.Cu at (-47.8, 176.9)
- added R32: 220, Resistors_SMD:R_0805_HandSoldering, F.Cu at (-87.8, 160.6)
- added R33: 220, Resistors_SMD:R_0805_HandSoldering, F.Cu at (-56.5, 118.2)
- added R34: 220, Resistors_SMD:R_0805_HandSoldering, F.Cu at (-56.5, 107.5)
- added R35: 220, Resistors_SMD:R_0805_HandSoldering, F.Cu at (-75.1, 156.0)
- added R36: 220, Resistors_SMD:R_0805_HandSoldering, F.Cu at (-64.8, 152.2)
- added R37: 10K, Resistors_SMD:R_0805_HandSoldering, F.Cu at (-52.2, 182.1)
- added R38: 1K, Resistors_SMD:R_0805_HandSoldering, F.Cu at (-78.9, 157.4)
- added R39: 220, Resistors_SMD:R_0805_HandSoldering, F.Cu at (-61.9, 173.2)
- added R40: 220, Resistors_SMD:R_0805_HandSoldering, F.Cu at (-53.4, 183.6)
- added R41: 220, Resistors_SMD:R_0805_HandSoldering, F.Cu at (-46.5, 175.4)
- added R42: 20K, Resistors_SMD:R_0805_HandSoldering, F.Cu at (-84.1, 159.3)
- added R43: 220, Resistors_SMD:R_0805_HandSoldering, F.Cu at (-56.5, 124.2)
- added R44: 10K, Resistors_SMD:R_0805_HandSoldering, F.Cu at (-14.2, 115.0)
- added R45: 10K, Resistors_SMD:R_0805_HandSoldering, F.Cu at (-14.2, 97.0)
- added R46: 10K, Resistors_SMD:R_0805_HandSoldering, F.Cu at (14.2, 86.0)
- added R47: 10K, Resistors_SMD:R_0805_HandSoldering, F.Cu at (14.2, 88.0)
- added R48: 10K, Resistors_SMD:R_0805_HandSoldering, F.Cu at (14.2, 90.0)
- added R49: 10K, Resistors_SMD:R_0805_HandSoldering, F.Cu at (14.2, 92.0)
- added R50: 10K, Resistors_SMD:R_0805_HandSoldering, F.Cu at (14.2, 94.0)
- added R51: 220, Resistors_SMD:R_0805_HandSoldering, F.Cu at (46.7, 115.2)
- added R52: 4.7K, Resistors_SMD:R_0805_HandSoldering, F.Cu at (66.2, 103.2)
- added R53: 10K, Resistors_SMD:R_0805_HandSoldering, F.Cu at (64.2, 103.2)
- added R54: 220, Resistors_SMD:R_0805_HandSoldering, F.Cu at (44.7, 115.2)
- added R55: 220, Resistors_SMD:R_0805_HandSoldering, F.Cu at (56.7, 103.2)
- added R56: 1K, Resistors_SMD:R_0805_HandSoldering, F.Cu at (58.7, 103.2)
- added R57: 10K, Resistors_SMD:R_0805_HandSoldering, F.Cu at (37.2, 130.9)
- added R58: 10K, Resistors_SMD:R_0805_HandSoldering, F.Cu at (22.0, 115.2)
- added R59: 10K, Resistors_SMD:R_0805_HandSoldering, F.Cu at (24.0, 115.2)
- added R60: 10K, Resistors_SMD:R_0805_HandSoldering, F.Cu at (22.0, 131.2)
- added R61: 10K, Resistors_SMD:R_0805_HandSoldering, F.Cu at (26.0, 115.2)
- added R62: 10K, Resistors_SMD:R_0805_HandSoldering, F.Cu at (24.0, 131.2)
- added R63: 10K, Resistors_SMD:R_0805_HandSoldering, F.Cu at (26.0, 131.2)
- added R64: 10K, Resistors_SMD:R_0805_HandSoldering, F.Cu at (44.7, 130.9)
- added R65: 1K, Resistors_SMD:R_0805_HandSoldering, F.Cu at (50.2, 130.9)
- added R66: 1K, Resistors_SMD:R_0805_HandSoldering, F.Cu at (40.7, 115.2)
- added R67: 1K, Resistors_SMD:R_0805_HandSoldering, F.Cu at (42.7, 130.9)
- added R68: 1K, Resistors_SMD:R_0805_HandSoldering, F.Cu at (53.1, 41.0)
- added R69: 10K, Resistors_SMD:R_0805_HandSoldering, F.Cu at (-10.5, 146.2)
- added R70: 10K, Resistors_SMD:R_0805_HandSoldering, F.Cu at (10.5, 148.2)
- added R71: 10K, Resistors_SMD:R_0805_HandSoldering, F.Cu at (10.5, 146.2)
- added R72: 1K, Resistors_SMD:R_0805_HandSoldering, F.Cu at (10.5, 136.8)
- added R73: 1K, Resistors_SMD:R_0805_HandSoldering, F.Cu at (-10.5, 137.2)
- added R74: 10K, Resistors_SMD:R_0805_HandSoldering, F.Cu at (45.1, 154.8)
- added R75: 10K, Resistors_SMD:R_0805_HandSoldering, F.Cu at (48.3, 181.9)
- added R76: 10K, Resistors_SMD:R_0805_HandSoldering, F.Cu at (62.0, 173.1)
- added R77: 10K, Resistors_SMD:R_0805_HandSoldering, F.Cu at (46.5, 151.0)
- added R78: 10K, Resistors_SMD:R_0805_HandSoldering, F.Cu at (47.1, 149.1)
- added R79: 10K, Resistors_SMD:R_0805_HandSoldering, F.Cu at (47.8, 147.3)
- added R8: 10K, Resistors_SMD:R_0805_HandSoldering, F.Cu at (-18.2, 197.4)
- added R80: 49.9, Resistors_SMD:R_0805_HandSoldering, F.Cu at (76.4, 165.2)
- added R81: 49.9, Resistors_SMD:R_0805_HandSoldering, F.Cu at (81.2, 152.1)
- added R82: 49.9, Resistors_SMD:R_0805_HandSoldering, F.Cu at (77.1, 163.3)
- added R83: 49.9, Resistors_SMD:R_0805_HandSoldering, F.Cu at (80.5, 153.9)
- added R84: 1K, Resistors_SMD:R_0805_HandSoldering, F.Cu at (66.9, 176.6)
- added R85: 1.5K, Resistors_SMD:R_0805_HandSoldering, F.Cu at (71.4, 179.7)
- added R86: 100K, Resistors_SMD:R_0805_HandSoldering, F.Cu at (57.6, 190.3)
- added R87: 220, Resistors_SMD:R_0805_HandSoldering, F.Cu at (63.6, 174.3)
- added R88: 220, Resistors_SMD:R_0805_HandSoldering, F.Cu at (50.0, 183.1)
- added R89: 220, Resistors_SMD:R_0805_HandSoldering, F.Cu at (60.4, 193.1)
- added R9: 10K, Resistors_SMD:R_0805_HandSoldering, F.Cu at (-6.58, 196.9)
- added R90: 220, Resistors_SMD:R_0805_HandSoldering, F.Cu at (76.3, 183.2)
- added R91: 220, Resistors_SMD:R_0805_HandSoldering, F.Cu at (48.5, 145.4)
- added R92: 220, Resistors_SMD:R_0805_HandSoldering, F.Cu at (49.2, 143.5)
- added R93: 220, Resistors_SMD:R_0805_HandSoldering, F.Cu at (73.0, 180.9)
- added R94: 15K, Resistors_SMD:R_0805_HandSoldering, F.Cu at (61.8, 194.5)
- added R95: 15K, Resistors_SMD:R_0805_HandSoldering, F.Cu at (63.2, 195.9)
- added R96: 10K, Resistors_SMD:R_0805_HandSoldering, F.Cu at (-43.5, 26.8)
- added R97: 10K, Resistors_SMD:R_0805_HandSoldering, F.Cu at (37.7, 174.5)
- added R98: 4.7K, Resistors_SMD:R_0805_HandSoldering, F.Cu at (-60.8, 150.8)
- added R99: 4.7K, Resistors_SMD:R_0805_HandSoldering, F.Cu at (-58.8, 150.0)
- added S1: SW_NAVI, my-switches:SW_NAVI_JS5208, F.Cu at (7.50, 19.0)
- added S2: SW_PUSH, my-switches:SW_PBUTTON_TL330, F.Cu at (30.2, 19.0)
- added S3: SW_PUSH, my-switches:SW_PBUTTON_TL330, F.Cu at (-14.8, 19.0)
- added S4: SW_PUSH_RA, my-switches:SW_SPSW_TACT_RA, F.Cu at (-44.8, 20.8)
- added S5: SW_PUSH_RA, my-switches:SW_SPSW_TACT_RA, F.Cu at (-36.2, 13.5)
- added U13: 74HCT595, Housings_SSOP:TSSOP-16_4.4x5mm_Pitch0.65mm, F.Cu at (-27.5, 163.0)
- added U14: 74HCT595, Housings_SSOP:TSSOP-16_4.4x5mm_Pitch0.65mm, F.Cu at (-8.75, 168.5)
- added U15: 74HCT595, Housings_SSOP:TSSOP-16_4.4x5mm_Pitch0.65mm, F.Cu at (9.00, 168.0)
- added U16: 74HCT595, Housings_SSOP:TSSOP-16_4.4x5mm_Pitch0.65mm, F.Cu at (26.3, 161.0)
- added U17: LPC1769, my-housings-qfp:LQFP-100_14x14mm_Pitch0.5mm, F.Cu at (0.25, 107.0)
- added U18: FT232R, Housings_SSOP:SSOP-28_5.3x10.2mm_Pitch0.65mm, F.Cu at (44.7, 103.2)
- added U19: 74HCT4066, Housings_SSOP:TSSOP-14_4.4x5mm_Pitch0.65mm, F.Cu at (32.0, 115.2)
- added U20: MAX3241E, Housings_SSOP:SSOP-28_5.3x10.2mm_Pitch0.65mm, F.Cu at (56.2, 122.9)
- added U21: 74HCT4066, Housings_SSOP:TSSOP-14_4.4x5mm_Pitch0.65mm, F.Cu at (32.0, 131.2)
- added U22: PIC16F1847, Housings_SSOP:SSOP-20_5.3x7.2mm_Pitch0.65mm, F.Cu at (0.25, 145.0)
- added U23: 74HCT4066, Housings_SSOP:TSSOP-14_4.4x5mm_Pitch0.65mm, F.Cu at (55.6, 172.9)
- added U24: LM3526-L, Housings_SOIC:SOIC-8_3.9x4.9mm_Pitch1.27mm, F.Cu at (44.0, 178.9)
- added U25: DP83848, my-housings-qfp:PQFP48-14x14mm, F.Cu at (63.3, 157.4)
- added U26: MIC39100-3.3, TO_SOT_Packages_SMD:SOT-223, F.Cu at (46.0, 52.5)
- added U27: MCP1322, TO_SOT_Packages_SMD:SOT-23-5, F.Cu at (-43.5, 29.5)
- added U28: 74HCT4066, Housings_SSOP:TSSOP-14_4.4x5mm_Pitch0.65mm, F.Cu at (48.0, 168.0)
- added XA1: SD-SOCKET, my-connect:SD_Card_Receptacle, B.Cu at (54.5, 175.3)
- added XBT1: CR2032-SOCKET, my-connect:SOCKET-SMT-CR2032-KEYSTONE-3003, B.Cu at (54.8, 74.2)
- added Y1: 12MHz, my-crystals:Crystal_SMD_5032_2Pads, F.Cu at (-4.50, 94.0)
- added Y2: 32.768KHz, my-crystals:Crystal_SMD_3215_2Pads, F.Cu at (2.50, 94.0)
- added Y3: 50MHz, TO_SOT_Packages_SMD:SOT-23-5, F.Cu at (53.6, 157.9)
- C1, C2, C3, C4, C5, C6, C8, C9: footprint Capacitors_SMD:C_0805 -> Capacitors_SMD:C_0805_HandSoldering
- C10, C11, C12: value 0.1uF -> 18pF; footprint Capacitors_SMD:C_0805 -> Capacitors_SMD:C_0805_HandSoldering
- C7: value 0.1uF -> 0.001uF; footprint Capacitors_SMD:C_0805 -> Capacitors_SMD:C_0805_HandSoldering
- J10: value BOXHDR2x3 -> HDR-1x9; footprint Pin_Headers:Pin_Header_Straight_2x05 -> my-connect:PHDR-RA-SMT-1x9; moved to B.Cu
- J3, J4, J6, J8: value BOXHDR2x5 -> BOXHDR-2x5; footprint Pin_Headers:Pin_Header_Straight_2x05 -> my-connect:SHDR-SMT-2x5
- J9: value CONN_01X06 -> HDR-1x6; footprint Pin_Headers:Pin_Header_Straight_1x06 -> my-connect:PHDR-RA-SMT-1x6; moved to B.Cu
- R1: value 4.7K -> 1K; footprint Resistors_SMD:R_0805 -> Resistors_SMD:R_0805_HandSoldering
- R2, R3, R4, R5, R6, R7: value 4.7K -> 10K; footprint Resistors_SMD:R_0805 -> Resistors_SMD:R_0805_HandSoldering
- U1: value LPC1769FBD100 -> 74HCT4066; footprint Housings_QFP:TQFP-100_14x14mm_Pitch0.5mm -> Housings_SSOP:TSSOP-14_4.4x5mm_Pitch0.65mm
- U10, U11, U12: value 74HC595 -> 74HCT4066; footprint Housings_SSOP:SSOP-16_5.3x6.2mm_Pitch0.65mm -> Housings_SSOP:TSSOP-14_4.4x5mm_Pitch0.65mm
- U2: value FT232RL -> 74HCT4066; footprint Housings_SSOP:SSOP-28_5.3x10.2mm_Pitch0.65mm -> Housings_SSOP:TSSOP-14_4.4x5mm_Pitch0.65mm
- U3, U8: value 74xx125 -> 74HCT4066
- U4, U5: value 74xx125 -> SN75176B; footprint Housings_SSOP:TSSOP-14_4.4x5mm_Pitch0.65mm -> Housings_SOIC:SOIC-8_3.9x4.9mm_Pitch1.27mm
- U6: value 75LBC176 -> MAX3241E; footprint Housings_SOIC:SOIC-8_3.9x4.9mm_Pitch1.27mm -> Housings_SSOP:SSOP-28_5.3x10.2mm_Pitch0.65mm
- U7: value 75LBC176 -> TJA1040
- U9: value 74HC595 -> MAX3241E; footprint Housings_SSOP:SSOP-16_5.3x6.2mm_Pitch0.65mm -> Housings_SSOP:SSOP-28_5.3x10.2mm_Pitch0.65mm
- moved R1 350.9 mm to (-22.2, 208.2), turned to 340 degrees
- moved R2 337.8 mm to (-20.3, 203.0), turned to 160 degrees
- moved C11 289.0 mm to (-6.50, 89.8), turned to 90 degrees
- moved J3 283.8 mm to (-23.8, 234.2), turned to 350 degrees
- moved R3 282.4 mm to (21.9, 204.6), turned to 20 degrees
- moved C10 281.5 mm to (-2.50, 89.8), turned to 90 degrees
- moved R4 277.3 mm to (23.3, 208.4), turned to 200 degrees
- moved C12 274.3 mm to (4.50, 89.8), turned to 90 degrees
- moved U3 268.2 mm to (-16.6, 192.4), turned to 340 degrees
- moved C6 261.9 mm to (-48.5, 197.6), turned to 320 degrees
- moved U12 258.1 mm to (-40.0, 133.8)
- moved C9 254.0 mm to (-49.8, 199.1), turned to 320 degrees
- moved C5 250.8 mm to (-34.1, 208.1), turned to 160 degrees
- moved U11 248.0 mm to (-40.0, 143.2)
- moved J4 246.8 mm to (-57.1, 220.4), turned to 330 degrees
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Connections:
- net /squid-logic/CFG0 renamed Net-(U9-Pad15)
- net /squid-logic/CFG4 renamed Net-(U9-Pad4)
- net /squid-logic/CFG5 renamed Net-(U9-Pad5)
- C1 pad 2: GND -> Net-(C1-Pad2)
- C10 pad 2: Net-(C10-Pad2) -> GND
- C11 pad 1: GND -> Net-(C11-Pad1)
- C11 pad 2: Net-(C11-Pad2) -> GND
- C12 pad 1: GND -> Net-(C12-Pad1)
- C12 pad 2: Net-(C12-Pad2) -> GND
- C2 pad 2: GND -> Net-(C2-Pad2)
- C3 pad 1: Net-(C3-Pad1) -> GND
- C4 pad 1: Net-(C4-Pad1) -> GND
- C7 pad 1: GND -> Net-(C7-Pad1)
- C7 pad 2: Net-(C7-Pad2) -> GND
- C9 pad 1: Net-(C9-Pad1) -> GND
- J10 pad 1: /CPU/COM3_MISO -> Net-(J10-Pad1)
- J10 pad 2: +5V -> GND
- J10 pad 3: /CPU/COM3_SCLK -> Net-(J10-Pad3)
- J10 pad 4: /CPU/COM3_MOSI -> /COM3, PROG/TCK
- J10 pad 5: /CPU/COM3_SSEL -> Net-(J10-Pad5)
- J10 pad 6: GND -> /COM3, PROG/TDO
- J10 pad 7: (no net) -> /COM3, PROG/TDI
- J10 pad 8: (no net) -> Net-(J10-Pad8)
- J10 pad 9: (no net) -> /COM3, PROG/TMS
- J3 pad 2: /Inputs/COM0B_DSR -> Net-(J3-Pad2)
- J3 pad 3: /Inputs/COM0B_RXD -> Net-(J3-Pad3)
- J3 pad 4: /Inputs/COM0B_RTS -> Net-(J3-Pad4)
- J3 pad 5: /Inputs/COM0B_TXD -> Net-(J3-Pad5)
- J3 pad 6: /Inputs/COM0B_CTS -> Net-(J3-Pad6)
- J3 pad 7: /Inputs/COM0B_DTR -> Net-(J3-Pad7)
- J4 pad 3: Net-(IC2-Pad6) -> Net-(J4-Pad3)
- J4 pad 4: Net-(IC2-Pad9) -> Net-(J4-Pad4)
- J4 pad 5: Net-(IC2-Pad10) -> Net-(J4-Pad5)
- J4 pad 6: Net-(IC2-Pad7) -> Net-(J4-Pad6)
- J6 pad 2: Net-(J6-Pad2) -> Net-(J25-Pad4)
- J6 pad 3: Net-(IC3-Pad6) -> Net-(J25-Pad3)
- J6 pad 4: Net-(IC3-Pad9) -> Net-(J25-Pad2)
- J6 pad 5: Net-(IC3-Pad10) -> Net-(J25-Pad4)
- J6 pad 8: Net-(J6-Pad8) -> +5V
- J6 pad 9: GND -> Net-(J25-Pad4)
- J8 pad 1: +5V -> Net-(J12-Pad2)
- J8 pad 10: /CPU/COM3_SSEL -> /COM3, PROG/~COM3_SSEL
- J8 pad 5: /CPU/COM3_SCL -> /COM3, PROG/COM3_SCL
- J8 pad 6: /CPU/COM3_SDA -> /COM3, PROG/COM3_SDA
- J8 pad 7: /CPU/COM3_MISO -> /COM3, PROG/COM3_MISO
- J8 pad 8: /CPU/COM3_MOSI -> /COM3, PROG/COM3_MOSI
- J8 pad 9: /CPU/COM3_SCLK -> /COM3, PROG/COM3_SCLK
- J9 pad 1: /CPU/COM3_SCL -> /COM3, PROG/COM3_SCL
- J9 pad 2: /CPU/COM3_SDA -> /COM3, PROG/COM3_SDA
- J9 pad 3: +5V -> Net-(J12-Pad2)
- J9 pad 5: /CPU/COM3_SCL -> /COM3, PROG/COM3_SCL
- J9 pad 6: /CPU/COM3_SDA -> /COM3, PROG/COM3_SDA
- R1 pad 1: +5V -> /CFG3
- R1 pad 2: /Inputs/COM0_ENA_TTL -> Net-(Q1-PadB)
- R2 pad 1: Net-(R2-Pad1) -> +3V3
- R2 pad 2: GND -> Net-(Q1-PadC)
- R3 pad 1: /CPU/COM1_TXDL -> /CFG4
- R4 pad 1: Net-(R4-Pad1) -> +3V3
- R4 pad 2: GND -> Net-(R4-Pad2)
- R5 pad 1: +5V -> Net-(R5-Pad1)
- R5 pad 2: /com1/nCOM1B_EN -> GND
- R6 pad 1: +5V -> Net-(R6-Pad1)
- R6 pad 2: /com1/nCOM1C_EN -> GND
- R7 pad 1: +5V -> /COM1/COM1_TXDL
- R7 pad 2: /com2/nCOM2B_EN -> GND
- U1 pad 1: Net-(U1-Pad1) -> Net-(R6-Pad1)
- U1 pad 13: (no net) -> /CFG4
- U1 pad 14: Net-(U1-Pad14) -> +5V
- U1 pad 2: Net-(U1-Pad2) -> /COM1/COM1_RTSL
- U1 pad 3: Net-(U1-Pad3) -> /COM1/COM1_RTSL
- U1 pad 4: Net-(U1-Pad4) -> Net-(R4-Pad2)
- U1 pad 5: Net-(U1-Pad5) -> /CFG4
- U1 pad 6: /CPU/COM3_RXD -> Net-(U1-Pad6)
- U1 pad 7: /CPU/COM3_TXD -> GND
- U10 pad 1: /squid-logic/CFG9 -> /COM3, PROG/COM3_SCL
- U10 pad 10: /squid-logic/nSHIFT_RESET -> /COM3, PROG/COM3_MOSI
- U10 pad 11: /squid-logic/SHIFT_CLK -> /COM3, PROG/COM3_MOSI
- U10 pad 12: /squid-logic/SHIFT_LOAD -> /CFG13
- U10 pad 13: /squid-logic/nSHIFT_OE -> /CFG13
- U10 pad 14: /squid-logic/CFG7 -> +5V
- U10 pad 2: /squid-logic/CFG10 -> /COM3, PROG/COM3_SCL
- U10 pad 3: /squid-logic/CFG11 -> /COM3, PROG/COM3_SDA
- U10 pad 4: /squid-logic/CFG12 -> /COM3, PROG/COM3_SDA
- U10 pad 5: /squid-logic/CFG13 -> /CFG13
- U10 pad 6: /squid-logic/CFG14 -> /CFG13
- U10 pad 7: /squid-logic/CFG15 -> GND
- U10 pad 8: GND -> /COM3, PROG/COM3_MISO
- U10 pad 9: Net-(U10-Pad9) -> /COM3, PROG/COM3_MISO
- U11 pad 1: /squid-logic/CFG17 -> /COM3, PROG/COM3_SCLK
- U11 pad 10: /squid-logic/nSHIFT_RESET -> /COM3, PROG/COM3_SCLK
- U11 pad 11: /squid-logic/SHIFT_CLK -> /COM3, PROG/TCK
- U11 pad 12: /squid-logic/SHIFT_LOAD -> /CFG16
- U11 pad 13: /squid-logic/nSHIFT_OE -> /CFG13
- U11 pad 14: /squid-logic/CFG15 -> +5V
- U11 pad 2: /squid-logic/CFG18 -> /COM3, PROG/COM3_SCLK
- U11 pad 3: /squid-logic/CFG19 -> /COM3, PROG/~COM3_SSEL
- U11 pad 4: /squid-logic/CFG20 -> /COM3, PROG/~COM3_SSEL
- U11 pad 5: /squid-logic/CFG21 -> /CFG13
- U11 pad 6: /squid-logic/CFG22 -> /CFG16
- U11 pad 7: /squid-logic/CFG23 -> GND
- U11 pad 8: GND -> /COM3, PROG/~COM3_SSEL
- U11 pad 9: Net-(U11-Pad9) -> /COM3, PROG/TMS
- U12 pad 1: /squid-logic/CFG25 -> /COM3, PROG/COM3_SCL
- U12 pad 10: /squid-logic/nSHIFT_RESET -> /COM3, PROG/COM3_SDA
- U12 pad 11: /squid-logic/SHIFT_CLK -> /COM3, PROG/~SRST
- U12 pad 12: /squid-logic/SHIFT_LOAD -> /CFG16
- U12 pad 13: /squid-logic/nSHIFT_OE -> /CFG16
- U12 pad 14: Net-(U12-Pad14) -> +5V
- U12 pad 2: /squid-logic/CFG26 -> /COM3, PROG/~TRST
- U12 pad 3: /squid-logic/CFG27 -> /COM3, PROG/COM3_MOSI
- U12 pad 4: /squid-logic/CFG28 -> /COM3, PROG/TDI
- U12 pad 5: /squid-logic/CFG29 -> /CFG16
- U12 pad 6: /squid-logic/CFG30 -> /CFG16
- U12 pad 7: /squid-logic/CFG31 -> GND
- U12 pad 8: GND -> /COM3, PROG/COM3_MISO
- U12 pad 9: Net-(U12-Pad9) -> /COM3, PROG/TDO
- U2 pad 1: /CPU/COM0_TXDL -> /COM1/COM1_RTSL
- U2 pad 11: /CPU/COM0_CTSL -> Net-(U2-Pad11)
- U2 pad 13: Net-(U2-Pad13) -> /CFG5
- U2 pad 14: Net-(U2-Pad14) -> +5V
- U2 pad 2: /Inputs/COM0_DTR -> /COM1/COM1C_RTSL
- U2 pad 3: /CPU/COM0_RTSL -> /COM1/COM1_DTRL
- U2 pad 4: Net-(U2-Pad4) -> /COM1/COM1C_DTR
- U2 pad 5: /CPU/COM0_RXDL -> /CFG5
- U2 pad 6: Net-(U2-Pad6) -> /CFG4
- U2 pad 8: (no net) -> Net-(R5-Pad1)
- U2 pad 9: /Inputs/COM0_DSR -> /COM1/COM1_DTRL
- U3 pad 1: /Inputs/COM0_ENA_TTL -> /COM1/COM1_DSRL
- U3 pad 10: /Inputs/COM0_ENA_TTL -> /COM1/COM1_RXDL
- U3 pad 11: /Inputs/COM0C_CTSL -> /COM1/COM1C_RXDL
- U3 pad 12: /CPU/COM0_CTSL -> /CFG5
- U3 pad 13: /Inputs/COM0_ENA_TTL -> /CFG5
- U3 pad 2: /Inputs/COM0C_RTSL -> /COM1/COM1C_DSR
- U3 pad 3: /CPU/COM0_RTSL -> /COM1/COM1_CTSL
- U3 pad 4: /Inputs/COM0_ENA_TTL -> /COM1/COM1C_CTSL
- U3 pad 5: /CPU/COM0_RXDL -> /CFG5
- U3 pad 6: /Inputs/COM0C_RXDL -> /CFG5
- U3 pad 8: /CPU/COM0_TXDL -> /COM1/COM1_TXDL
- U3 pad 9: /Inputs/COM0B_TXD -> /COM1/COM1C_TXD
- U4 pad 1: /com1/nCOM1B_EN -> Net-(U4-Pad1)
- U4 pad 2: /CPU/COM1_RTSL -> Net-(U4-Pad2)
- U4 pad 3: Net-(R4-Pad1) -> Net-(R5-Pad1)
- U4 pad 4: /com1/nCOM1B_EN -> /COM1/COM1_TXDL
- U4 pad 5: /CPU/COM1_DTRL -> GND
- U4 pad 6: Net-(R2-Pad1) -> /COM1/RXB
- U4 pad 7: GND -> /COM1/RXA
- U4 pad 8: /com1/COM1C_DTRL -> +5V
- U5 pad 1: /com1/nCOM1C_EN -> /COM1/COM1_RXDL
- U5 pad 2: /CPU/COM1_RTSL -> Net-(R4-Pad2)
- U5 pad 3: /com1/COM1C_RTSL -> Net-(R6-Pad1)
- U5 pad 4: /com1/nCOM1C_EN -> /COM1/COM1_TXDL
- U5 pad 5: /com1/COM1C_RXDL -> GND
- U5 pad 6: /CPU/COM1_RXDL -> /COM1/TXB
- U5 pad 7: GND -> /COM1/TXA
- U5 pad 8: /com1/COM1C_TXDL -> +5V
- U6 pad 1: Net-(U6-Pad1) -> Net-(C2-Pad1)
- U6 pad 2: Net-(U6-Pad2) -> Net-(C2-Pad2)
- U6 pad 3: Net-(R2-Pad1) -> Net-(C4-Pad2)
- U6 pad 4: /CPU/COM1_TXDL -> Net-(J3-Pad1)
- U6 pad 5: GND -> Net-(J3-Pad2)
- U6 pad 6: Net-(P6-Pad4) -> Net-(J3-Pad3)
- U6 pad 7: Net-(P6-Pad5) -> Net-(J3-Pad6)
- U6 pad 8: +5V -> Net-(J3-Pad8)
- U7 pad 1: /CPU/COM1_RXDL -> /COM2-CAN/CAN_TD
- U7 pad 2: Net-(R4-Pad1) -> GND
- U7 pad 3: Net-(R4-Pad1) -> +5V
- U7 pad 4: /CPU/COM1_TXDL -> /COM2-CAN/CAN_RD
- U7 pad 5: GND -> Net-(C7-Pad1)
- U7 pad 6: Net-(P6-Pad2) -> Net-(J25-Pad3)
- U7 pad 7: Net-(P6-Pad1) -> Net-(J25-Pad2)
- U7 pad 8: +5V -> /CFG12
- U8 pad 1: /com2/nCOM2B_EN -> /COM2-CAN/COM2B_RTSL
- U8 pad 10: /com2/nCOM2B_EN -> /COM2-CAN/COM2_CTSL
- U8 pad 11: /CPU/COM2_CTSL -> /COM2-CAN/COM2B_CTSL
- U8 pad 12: Net-(U8-Pad12) -> /CFG9
- U8 pad 13: /com2/nCOM2B_EN -> /CFG9
- U8 pad 2: /CPU/COM2_RTSL -> /COM2-CAN/COM2_RTSL
- U8 pad 3: /com2/COM2B_RTSL -> /COM2-CAN/COM2B_TXD
- U8 pad 4: /com2/nCOM2B_EN -> /COM2-CAN/COM2_TXDL
- U8 pad 5: Net-(U8-Pad5) -> /CFG9
- U8 pad 6: /CPU/COM2_RXDL -> /CFG9
- U8 pad 8: /com2/COM2B_TXDL -> /COM2-CAN/COM2_RXDL
- U8 pad 9: /CPU/COM2_TXDL -> /COM2-CAN/COM2B_RXDL
- U9 pad 1: /squid-logic/CFG1 -> Net-(C6-Pad1)
- U9 pad 10: /squid-logic/nSHIFT_RESET -> Net-(J4-Pad5)
- U9 pad 11: /squid-logic/SHIFT_CLK -> Net-(U9-Pad11)
- U9 pad 12: /squid-logic/SHIFT_LOAD -> Net-(U9-Pad12)
- U9 pad 13: /squid-logic/nSHIFT_OE -> /COM2-CAN/COM2_TXDL
- U9 pad 14: /squid-logic/SHIFT_IN -> /COM2-CAN/COM2_RTSL
- U9 pad 16: VCC -> /COM2-CAN/COM2_CTSL
- U9 pad 2: /squid-logic/CFG2 -> Net-(C6-Pad2)
- U9 pad 3: /squid-logic/CFG3 -> Net-(C9-Pad2)
- U9 pad 6: /squid-logic/CFG6 -> Net-(J4-Pad3)
- U9 pad 7: /squid-logic/CFG7 -> Net-(J4-Pad6)
- U9 pad 8: GND -> Net-(U9-Pad8)
- U9 pad 9: Net-(U9-Pad9) -> Net-(J4-Pad4)
Other:
- board size 177.3 x 205 mm -> 216.7 x 240 mm
- board text added: "+3.3V"
- board text added: "+5V"
- board text added: "RS232"
- board text added: "TTL"

Commit message: parts placement, draft 2, straight alignment
Parts:
- J18: footprint my-connect:MINIDIN-STR-THRU-6 -> my-connect:MINIDIN-RA-THRU-6
- S3: footprint my-switches:SW_PBUTTON_TL330 -> SW_PBUTTON_TL330
- moved C21 220.4 mm to (257.8, 216.8), turned to 0 degrees
- moved C47 217.1 mm to (243.0, 145.2), turned to 180 degrees
- moved U24 216.4 mm to (257.8, 212.8), turned to 0 degrees
- moved C50 216.1 mm to (243.0, 153.2), turned to 180 degrees
- moved U19 213.7 mm to (243.0, 149.2), turned to 0 degrees
- moved U21 212.7 mm to (243.1, 157.2), turned to 0 degrees
- moved U13 212.2 mm to (182.0, 197.0)
- moved R32 211.8 mm to (120.0, 201.5), turned to 0 degrees
- moved C15 211.5 mm to (260.2, 156.0), turned to 0 degrees
- moved R75 211.1 mm to (257.8, 208.8), turned to 0 degrees
- moved Q18 211.1 mm to (218.0, 178.2)
- moved R72 211.1 mm to (218.0, 175.5)
- moved C48 210.6 mm to (257.8, 154.0), turned to 180 degrees
- moved C30 210.4 mm to (243.0, 234.0), turned to 0 degrees
- moved R58 210.4 mm to (229.0, 152.8), turned to 0 degrees
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Other:
- outline, holes or cut-outs redrawn
- board text removed: "+3.3V"
- board text removed: "+5V"
- board text removed: "RS232"
- board text removed: "TTL"
